File: Hardware/Schematic.sch (EAGLE design)
At the start: 103 parts, among them IC1 BQ25180YBGR_BQ25180YBGR, IC2 RT6160AWSC_RT6160AWSC, IC3 BMA423_BMA423, IC4 DRV2605YZFR_DRV2605YZFR, J1 TC2030-IDC_TC2030-IDC, J2 503480-2400, J4 KH-TYPE-C-16P, Q1 20V/4.2A/52mΩ/1.4W, Q3 SI1308EDL-T1-GE3, U3 MAX17048G+T10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

Commit message: schematic upate
Parts:
- C23: value 10uF -> 0.1uF
- C24: value 0.1uF -> 10uF
- IC3: value BMA423_BMA423 -> BMA421_BMA421; device InkTime_v5:BMA423_BMA423 -> InkTime_v5:BMA421_BMA421
Changed lines of the file:
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@@
 <part name="IC2" library="InkTime_v5" deviceset="RT6160AWSC_RT6160AWSC" device=""/>
 <part name="U3" library="InkTime_v5" deviceset="ESP32_C6_LIBRARY_MAX17048G+T10" device="" value="MAX17048G+T10"/>
-<part name="IC3" library="InkTime_v5" deviceset="BMA423_BMA423" device=""/>
+<part name="IC3" library="InkTime_v5" deviceset="BMA421_BMA421" device=""/>
 <part name="IC4" library="InkTime_v5" deviceset="DRV2605YZFR_DRV2605YZFR" device=""/>
 <part name="Q1" library="InkTime_v5" deviceset="ESP32_C6_LIBRARY_4_ESP32_WROVER_SPARKFUN-DISCRETESEMI_MOSFET_PCH" device="-DMG2305UX-7" value="20V/4.2A/52mΩ/1.4W"/>
@@
 <part name="R4" library="InkTime_v5" deviceset="CPF0201D7K68C1_CPF0201D7K68C1" device="" value="0"/>
 <part name="R2" library="InkTime_v5" deviceset="CPF0201D7K68C1_CPF0201D7K68C1" device="" value="0"/>
-<part name="C24" library="InkTime_v5" deviceset="GRM011R60J152KE01L_2_GRM011R60J152KE01L" device="" value="0.1uF"/>
-<part name="C23" library="InkTime_v5" deviceset="ESP32_C6_LIBRARY_1_ESP32_WROVER_EAGLE-LTSPICE_C" device="C0402" value="10uF"/>
+<part name="C24" library="InkTime_v5" deviceset="GRM011R60J152KE01L_2_GRM011R60J152KE01L" device="" value="10uF"/>
+<part name="C23" library="InkTime_v5" deviceset="ESP32_C6_LIBRARY_1_ESP32_WROVER_EAGLE-LTSPICE_C" device="C0402" value="0.1uF"/>
 <part name="GND6" library="InkTime_v5" deviceset="HECTOR_WATCH_2_GND" device="" value="GND"/>
 <part name="GND7" library="InkTime_v5" deviceset="HECTOR_WATCH_2_GND" device=""/>
